File: usb3_fiber.kicad_pcb (KiCad board)
At the start: 4 copper layers, 75 x 40 mm, 64 parts, among them J1 U77A16382001, J2 UE76A202000T, J3 10118194-0001LF, J4 GSB4211311WEU, J5 GSB3111311HR, Q1 MMBT3906, U1 MCP2221AT-I/ML, U2 DS100BR111SQE/NOPB, U4 LD1086D2T33TR

Commit message: ci: main-release workflow + build-time revision/GIT_HASH provenance (#5)
* Add main-release CI + build-time revision/GIT_HASH provenance

Phase 4 (folds in Phase 2 provenance):

- Define ${REVISION}/${GIT_HASH} project text variables and reference
  them in the schematic + PCB title blocks (rev field + git-hash
  comment). Defaults are placeholders; CI overwrites them at build time.
- scripts/build_release.sh: inject REVISION/GIT_HASH into the project
  text variables (build-time only, never committed back), then export
  the full package — gerbers, drill, CPL, STEP, schematic PDF, grouped
  BOM, and top/bottom assembly drawings.
- .github/workflows/main-release.yml: manual workflow_dispatch release.
  Computes the next alpha revision from the latest GitHub Release
  (source of truth), builds in the KiCad 10 container, and publishes a
  GitHub Release with the packaged artifacts.

Bottom-silkscreen provenance text is intentionally left to be placed in
KiCad (blind coordinate placement risks silk-over-pad overlaps) — once
added referencing the same variables, CI fills it automatically.

Co-Authored-By: Claude Opus 4.8 <noreply@anthropic.com>
Claude-Session: https://claude.ai/code/session_012vRW6hhKX7UfnTmWpMyfnj

* added silk for project name, revision and commit hash

* ci: echo ERC/DRC/BOM report detail into run log + job summary

Add emit_report helper to dev-checks so the full erc.rpt/drc.rpt/
bom_check.txt contents appear in the run log (collapsible) and the job
summary, making the baseline readable without downloading the artifact.

Co-Authored-By: Claude Opus 4.8 <noreply@anthropic.com>
Claude-Session: https://claude.ai/code/session_012vRW6hhKX7UfnTmWpMyfnj

* ci: bump actions to Node 24 majors (checkout/upload/download @v6)

Clear the 'Node.js 20 is deprecated' runner annotation by moving
actions/checkout, actions/upload-artifact, and actions/download-artifact
from @v4 (Node 20) to @v6 (Node 24) in both workflows.

Co-Authored-By: Claude Opus 4.8 <noreply@ant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
Other:
- board text added: "${PROJECTNAME} Rev: ${REVISION} Commit: ${GIT_HASH}"
Changed lines of the file:
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@@
 		(title "USB 3.0 to SFP+ Board")
 		(date "2026-03-13")
-		(rev "1")
+		(rev "${REVISION}")
+		(comment 1 "Git: ${GIT_HASH}")
 	)
 	(layers
@@
 		)
 	)
+	(property "GIT_HASH" "local")
+	(property "REVISION" "DEV")
 	(footprint "MountingHole:MountingHole_2.7mm_M2.5"
 		(locked yes)
@@
 		(layer "Edge.Cuts")
 	)
+	(gr_text "${PROJECTNAME}\nRev: ${REVISION} \nCommit: ${GIT_HASH}"
+		(at 180 105 0)
+		(layer "B.SilkS" knockout)
+		(effects
+			(font
+				(size 2 2)
+				(thickness 0.5)
+				(bold yes)
+			)
+			(justify left bottom mirror)
+		)
+	)
 	(gr_text "FABRICATION SPECIFICATION\n========================================\nProject: USB3 Fiber Link\n\nGENERAL\n  Layers: 4 (TOP / GND / PWR / BOTTOM)\n  Material: FR4, Standard Tg (150-160C)\n  Finished Thickness: 62 mil (1.575mm) +/- 10%\n  Surface Finish: ENIG (1u\")\n  Solder Mask: Green, both sides\n  Silkscreen: White, both sides\n  IPC Class: 2\n\nSTACKUP\n  F.Cu:   1 oz (0.035mm) - Signal\n  Prepreg: 0.21mm (7628, Er=4.5)\n  In1.Cu: 0.5 oz (0.0175mm) - GND Plane\n  Core:   1.03mm (Er=4.5)\n  In2.Cu: 0.5 oz (0.0175mm) - PWR Plane\n  Prepreg: 0.21mm (7628, Er=4.5)\n  B.Cu:   1 oz (0.035mm) - Signal\n\nCONTROLLED IMPEDANCE\n  USB3 SuperSpeed: 100 ohm diff, 50 ohm SE\n  SFP+ CML:       100 ohm diff, 50 ohm SE\n  USB2 High-Speed: 90 ohm diff, 45 ohm SE\n  Tolerance: +/-10% (+/-5 ohm if <= 50 ohm)\n  Verify trace width with fab stackup calculator\n\nMINIMUM FEATURES (JLCPCB 4-layer 1oz)\n  Track width:     0.10mm (4 mil)\n  Track spacing:   0.10mm (4 mil)\n  Via drill/dia:   0.30mm / 0.50mm\n  Annular ring:    0.10mm\n  Hole-to-hole:    0.25mm\n  Copper-to-edge:  0.50mm\n  Solder mask bridge: 0.10mm\n  Mask-to-trace:   0.09mm\n\nVIA PLUGGING\n  Fill vias with soldermask (opaque)\n  Max via diameter for plugging: 0.5mm\n\nNOTES\n  1. All dimensions in mm unless noted\n  2. Panelize per fab requirements\n  3. No blind/buried vias required"
 		(at 44 90 0)
@@
 	)
 	(segment
-		(start 132.09 100.5375)
-		(end 131.79 100.2375)
+		(start 127.56 104.5375)
+		(end 128.31 105.2875)
 		(width 0.2)
 		(layer "F.Cu")
-		(net "/SSRX-")
+		(net "/SSTX-")
 	)
 	(segment
-		(start 132.12 100.5375)
-		(end 132.09 100.5375)
+		(start 119.6 104.5375)
+		(end 127.56 104.5375)
 		(width 0.2)
 		(layer "F.Cu")
-		(net "/SSRX-")
+		(net "/SSTX-")
 	)
 	(segment
-		(start 129.494314 98.5375)
-		(end 128.31 98.5375)
+		(start 131.354999 102.7375)
+		(end 130.86 102.7375)
 		(width 0.2)
 		(layer "F.Cu")
-		(net "/SSRX-")
+		(net "/SSTX-")
 	)
 	(segment
-		(start 131.194314 100.2375)
-		(end 129.494314 98.5375)
+		(start 131.654999 103.0375)
+		(end 131.354999 102.7375)
 		(width 0.2)
 		(layer "F.Cu")
-		(net "/SSRX-")
+		(net "/SSTX-")
 	)
 	(segment
-		(start 131.79 100.2375)
-		(end 131.194314 100.2375)
+		(start 132.12 103.0375)
+		(end 131.654999 103.0375)
 		(width 0.2)
 		(layer "F.Cu")
-		(net "/SSRX-")
+		(net "/SSTX-")
 	)
 	(segment
-		(start 127.56 104.5375)
-		(end 128.31 105.2875)
+		(start 119.1 105.0375)
+		(end 119.6 104.5375)
 		(width 0.2)
 		(layer "F.Cu")
@@
 	)
 	(segment
-		(start 119.6 104.5375)
-		(end 127.56 104.5375)
+		(start 130.86 102.7375)
+		(end 128.31 105.2875)
 		(width 0.2)
 		(layer "F.Cu")
@@
 	)
 	(segment
-		(start 131.354999 102.7375)
-		(end 130.86 102.7375)
+		(start 132.09 100.5375)
+		(end 131.79 100.2375)
 		(width 0.2)
 		(layer "F.Cu")
-		(net "/SSTX-")
+		(net "/SSRX-")
 	)
 	(segment
-		(start 131.654999 103.0375)
-		(end 131.354999 102.7375)
+		(start 132.12 100.5375)
+		(end 132.09 100.5375)
 		(width 0.2)
 		(layer "F.Cu")
-		(net "/SSTX-")
+		(net "/SSRX-")
 	)
 	(segment
-		(start 132.12 103.0375)
-		(end 131.654999 103.0375)
+		(start 129.494314 98.5375)
+		(end 128.31 98.5375)
 		(width 0.2)
 		(layer "F.Cu")
-		(net "/SSTX-")
+		(net "/SSRX-")
 	)
 	(segment
-		(start 119.1 105.0375)
-		(end 119.6 104.5375)
+		(start 131.194314 100.2375)
+		(end 129.494314 98.5375)
 		(width 0.2)
 		(layer "F.Cu")
-		(net "/SSTX-")
+		(net "/SSRX-")
 	)
 	(segment
-		(start 130.86 102.7375)
-		(end 128.31 105.2875)
+		(start 131.79 100.2375)
+		(end 131.194314 100.2375)
 		(width 0.2)
 		(layer "F.Cu")
-		(net "/SSTX-")
+		(net "/SSRX-")
+	)
+	(segment
+		(start 121.35 119.5375)
+		(end 121.35 118.0375)
+		(width 0.2)
+		(layer "F.Cu")
+		(net "/D-")
+	)
+	(via
+		(at 121.35 119.5375)
+		(size 0.6)
+		(drill 0.3)
+		(layers "F.Cu" "B.Cu")
+		(free yes)
+		(capping no)
+		(covering
+			(front no)
+			(back no)
+		)
+		(plugging
+			(front no)
+			(back no)
+		)
+		(filling no)
+		(net "/D-")
+	)
+	(segment
+		(start 121.35 114.0375)
+		(end 121.35 115.5375)
+		(width 0.2)
+		(layer "F.Cu")
+		(net "/D+")
+	)
+	(via
+		(at 121.35 114.0375)
+		(size 0.6)
+		(drill 0.3)
+		(layers "F.Cu" "B.Cu")
+		(free yes)
+		(capping no)
+		(covering
+			(front no)
+			(back no)
+		)
+		(plugging
+			(front no)
+			(back no)
+		)
+		(filling no)
+		(net "/D+")
 	)
 	(segment
@@
 	)
 	(segment
-		(start 117.45 116.0845)
-		(end 119.403 118.0375)
-		(width 0.2)
-		(layer "F.Cu")
-		(net "/D-_2")
-	)
-	(segment
-		(start 119.403 118.0375)
-		(end 120.05 118.0375)
-		(width 0.2)
-		(layer "F.Cu")
-		(net "/D-_2")
-	)
-	(segment
-		(start 116.575 116.0845)
-		(end 117.45 116.0845)
-		(width 0.2)
-		(layer "F.Cu")
-		(net "/D-_2")
-	)
-	(segment
-		(start 119.947 115.4345)
-		(end 120.05 115.5375)
-		(width 0.2)
-		(layer "F.Cu")
-		(net "/D+_2")
-	)
-	(segment
-		(start 116.575 115.4345)
-		(end 119.947 115.4345)
+		(start 137.95 103.3149)
+		(end 137.95 103.8875)
 		(width 0.2)
 		(layer "F.Cu")
-		(net "/D+_2")
+		(net "Net-(U2-MODE{slash}~{DONE})")
 	)
 	(segment
-		(start 121.35 114.0375)
-		(end 121.35 115.5375)
+		(start 137.95 103.8875)
+		(end 138.35 104.2875)
 		(width 0.2)
 		(layer "F.Cu")
-		(net "/D+")
+		(net "Net-(U2-MODE{slash}~{DONE})")
 	)
 	(via
-		(at 121.35 114.0375)
+		(at 138.35 104.2875)
 		(size 0.6)
 		(drill 0.3)
@@
 		)
 		(filling no)
-		(net "/D+")
+		(net "Net-(U2-MODE{slash}~{DONE})")
 	)
 	(segment
-		(start 121.35 119.5375)
-		(end 121.35 118.0375)
+		(start 119.947 115.4345)
+		(end 120.05 115.5375)
 		(width 0.2)
 		(layer "F.Cu")
-		(net "/D-")
+		(net "/D+_2")
 	)
-	(via
-		(at 121.35 119.5375)
-		(size 0.6)
-		(drill 0.3)
-		(layers "F.Cu" "B.Cu")
-		(free yes)
-		(capping no)
-		(covering
-			(front no)
-			(back no)
-		)
-		(plugging
-			(front no)
-			(back no)
-		)
-		(filling no)
-		(net "/D-")
+	(segment
+		(start 116.575 115.4345)
+		(end 119.947 115.4345)
+		(width 0.2)
+		(layer "F.Cu")
+		(net "/D+_2")
 	)
 	(segment
-		(start 137.95 103.3149)
-		(end 137.95 103.8875)
+		(start 117.45 116.0845)
+		(end 119.403 118.0375)
 		(width 0.2)
 		(layer "F.Cu")
-		(net "Net-(U2-MODE{slash}~{DONE})")
+		(net "/D-_2")
 	)
 	(segment
-		(start 137.95 103.8875)
-		(end 138.35 104.2875)
+		(start 119.403 118.0375)
+		(end 120.05 118.0375)
 		(width 0.2)
 		(layer "F.Cu")
-		(net "Net-(U2-MODE{slash}~{DONE})")
+		(net "/D-_2")
 	)
-	(via
-		(at 138.35 104.2875)
-		(size 0.6)
-		(drill 0.3)
-		(layers "F.Cu" "B.Cu")
-		(free yes)
-		(capping no)
-		(covering
-			(front no)
-			(back no)
-		)
-		(plugging
-			(front no)
-			(back no)
-		)
-		(filling no)
-		(net "Net-(U2-MODE{slash}~{DONE})")
+	(segment
+		(start 116.575 116.0845)
+		(end 117.45 116.0845)
+		(width 0.2)
+		(layer "F.Cu")
+		(net "/D-_2")
 	)
 	(zone
